File: lab01/zad2/zad2/zad2.sch (KiCad schematic (older format))
At the start: 7 parts

Commit message: lab01
Parts:
- RV?: value R_POT -> 10 kOhm
Connections:
- net at A?.7 (GND), RV?.3: no longer R?.2, R?.2
- net at A?.10 (A1): no longer D?.2 (A)
- net at R?.1, SW?.1 (A): now also A?.18 (D3); no longer A?.11 (A2)
- net at A?.17 (D2): now also D?.2 (A)
- net at A?.29 (GND): now also R?.2, R?.2
Other:
- moved on the sheet: D?, PC?, R?, RV?, SW?A
Changed lines of the file:
@@
 L local:PC PC?
 U 1 1 5E88DFB1
-P 2300 3550
-F 0 "PC?" H 2333 4215 50  0000 C CNN
-F 1 "PC" H 2333 4124 50  0000 C CNN
-F 2 "" H 2300 3550 50  0001 C CNN
-F 3 "" H 2300 3550 50  0001 C CNN
-	1    2300 3550
+P 2000 2500
+F 0 "PC?" H 2033 3165 50  0000 C CNN
+F 1 "PC" H 2033 3074 50  0000 C CNN
+F 2 "" H 2000 2500 50  0001 C CNN
+F 3 "" H 2000 2500 50  0001 C CNN
+	1    2000 2500
 	1    0    0    -1
 $EndComp
-Wire Wire Line
-	4250 3550 2900 3550
-Wire Wire Line
-	2900 3550 2900 3250
-Wire Wire Line
-	4250 3650 2900 3650
-Wire Wire Line
-	2900 3650 2900 3850
 $Comp
 L Device:LED D?
 U 1 1 5E87A2AD
-P 5550 4600
-F 0 "D?" V 5589 4483 50  0000 R CNN
-F 1 "LED" V 5498 4483 50  0000 R CNN
-F 2 "" H 5550 4600 50  0001 C CNN
-F 3 "~" H 5550 4600 50  0001 C CNN
-	1    5550 4600
+P 3700 4600
+F 0 "D?" V 3739 4483 50  0000 R CNN
+F 1 "LED" V 3648 4483 50  0000 R CNN
+F 2 "" H 3700 4600 50  0001 C CNN
+F 3 "~" H 3700 4600 50  0001 C CNN
+	1    3700 4600
 	0    -1   -1   0
 $EndComp
@@
 L Switch:SW_DPST_x2 SW?
 U 1 1 5E87AFAE
-P 7100 3700
-F 0 "SW?" H 7100 3935 50  0000 C CNN
-F 1 "SW_DPST_x2" H 7100 3844 50  0000 C CNN
-F 2 "" H 7100 3700 50  0001 C CNN
-F 3 "~" H 7100 3700 50  0001 C CNN
-	1    7100 3700
+P 3150 3500
+F 0 "SW?" H 3150 3735 50  0000 C CNN
+F 1 "SW_DPST_x2" H 3150 3644 50  0000 C CNN
+F 2 "" H 3150 3500 50  0001 C CNN
+F 3 "~" H 3150 3500 50  0001 C CNN
+	1    3150 3500
 	0    -1   -1   0
 $EndComp
@@
 L Device:R R?
 U 1 1 5E87BA0D
-P 7100 4850
-F 0 "R?" H 7170 4896 50  0000 L CNN
-F 1 "10 kOhm" H 7170 4805 50  0000 L CNN
-F 2 "" V 7030 4850 50  0001 C CNN
-F 3 "~" H 7100 4850 50  0001 C CNN
-	1    7100 4850
+P 3150 4850
+F 0 "R?" H 3220 4896 50  0000 L CNN
+F 1 "10 kOhm" H 3220 4805 50  0000 L CNN
+F 2 "" V 3080 4850 50  0001 C CNN
+F 3 "~" H 3150 4850 50  0001 C CNN
+	1    3150 4850
 	1    0    0    -1
-$EndComp
-Wire Wire Line
-	5250 4150 5700 4150
-$Comp
-L Device:R_POT RV?
-U 1 1 5E8714BC
-P 5850 4150
-F 0 "RV?" H 5781 4196 50  0000 R CNN
-F 1 "R_POT" H 5781 4105 50  0000 R CNN
-F 2 "" H 5850 4150 50  0001 C CNN
-F 3 "~" H 5850 4150 50  0001 C CNN
-	1    5850 4150
-	-1   0    0    -1
 $EndComp
 Wire Wire Line
 	4950 3150 5850 3150
 Wire Wire Line
-	5850 3150 5850 4000
+	5850 3150 5850 3650
 Wire Wire Line
-	5850 4300 5850 5250
-Wire Wire Line
-	5850 5250 5550 5250
-Wire Wire Line
-	7100 3150 7100 3500
-Wire Wire Line
-	7100 3900 7100 4350
-Wire Wire Line
-	7100 4350 7100 4700
-Connection ~ 7100 4350
-Wire Wire Line
-	7100 5000 7100 5250
-Wire Wire Line
-	5250 4350 7100 4350
-Wire Wire Line
-	5850 3150 7100 3150
-Connection ~ 5850 3150
-Wire Wire Line
-	5850 5250 7100 5250
-Connection ~ 5850 5250
+	3150 5000 3150 5250
 $Comp
 L Device:R R?
 U 1 1 5E897C7D
-P 5550 4900
-F 0 "R?" H 5620 4946 50  0000 L CNN
-F 1 "2.2 kOhm" H 5620 4855 50  0000 L CNN
-F 2 "" V 5480 4900 50  0001 C CNN
-F 3 "~" H 5550 4900 50  0001 C CNN
-	1    5550 4900
+P 3700 4900
+F 0 "R?" H 3770 4946 50  0000 L CNN
+F 1 "2.2 kOhm" H 3770 4855 50  0000 L CNN
+F 2 "" V 3630 4900 50  0001 C CNN
+F 3 "~" H 3700 4900 50  0001 C CNN
+	1    3700 4900
 	1    0    0    -1
 $EndComp
 Wire Wire Line
-	5550 5050 5550 5250
-Connection ~ 5550 5250
+	3700 5050 3700 5250
 Wire Wire Line
-	5550 5250 4850 5250
+	4850 5250 5850 5250
 Wire Wire Line
-	5250 4250 5550 4250
+	3150 3700 3150 3850
+$Comp
+L Device:R_POT RV?
+U 1 1 5E8714BC
+P 5850 3800
+F 0 "RV?" H 5781 3846 50  0000 R CNN
+F 1 "10 kOhm" H 5781 3755 50  0000 R CNN
+F 2 "" H 5850 3800 50  0001 C CNN
+F 3 "~" H 5850 3800 50  0001 C CNN
+	1    5850 3800
+	-1   0    0    -1
+$EndComp
 Wire Wire Line
-	5550 4250 5550 4450
+	5850 3950 5850 5250
+Wire Wire Line
+	4250 3550 4250 2200
+Wire Wire Line
+	4250 2200 2600 2200
+Wire Wire Line
+	2600 2800 4100 2800
+Wire Wire Line
+	4100 2800 4100 3650
+Wire Wire Line
+	4100 3650 4250 3650
+Wire Wire Line
+	3150 3050 3150 3300
+Wire Wire Line
+	4950 3150 4950 3050
+Connection ~ 4950 3150
+Wire Wire Line
+	3150 3050 4950 3050
+Connection ~ 3700 5250
+Wire Wire Line
+	3700 5250 3150 5250
+Wire Wire Line
+	3700 4450 3700 3750
+Wire Wire Line
+	3700 3750 4250 3750
+Wire Wire Line
+	3700 5250 4650 5250
+Wire Wire Line
+	4250 3850 3150 3850
+Connection ~ 3150 3850
+Wire Wire Line
+	3150 3850 3150 4700
+Wire Wire Line
+	5700 3800 5400 3800
+Wire Wire Line
+	5400 3800 5400 4150
+Wire Wire Line
+	5400 4150 5250 4150
 $EndSCHEMATC
