File: lab01/zad3/zad3/zad3.sch (KiCad schematic (older format))
At the start: 7 parts

Commit message: lab01
Parts:
- added C?: 4.7 uF, symbol Device:C
- added R?: 4.7 kOhm, symbol Device:R
- RV?: value R_POT -> 10 kOhm
Connections:
- net at A?.7 (GND), RV?.3: now also R?.2
- net at A?.11 (A2): now also C?.2, R?.1
- net at A?.24 (D9): now also C?.1
Changed lines of the file:
@@
 P 5850 3800
 F 0 "RV?" H 5781 3846 50  0000 R CNN
-F 1 "R_POT" H 5781 3755 50  0000 R CNN
+F 1 "10 kOhm" H 5781 3755 50  0000 R CNN
 F 2 "" H 5850 3800 50  0001 C CNN
 F 3 "~" H 5850 3800 50  0001 C CNN
@@
 Wire Wire Line
 	5400 4150 5250 4150
+$Comp
+L Device:R R?
+U 1 1 5E89D0D1
+P 4700 5900
+F 0 "R?" H 4770 5946 50  0000 L CNN
+F 1 "4.7 kOhm" H 4770 5855 50  0000 L CNN
+F 2 "" V 4630 5900 50  0001 C CNN
+F 3 "~" H 4700 5900 50  0001 C CNN
+	1    4700 5900
+	0    -1   -1   0
+$EndComp
+$Comp
+L Device:C C?
+U 1 1 5E89D73D
+P 4400 5900
+F 0 "C?" H 4515 5946 50  0000 L CNN
+F 1 "4.7 uF" H 4515 5855 50  0000 L CNN
+F 2 "" H 4438 5750 50  0001 C CNN
+F 3 "~" H 4400 5900 50  0001 C CNN
+	1    4400 5900
+	0    -1   -1   0
+$EndComp
+Wire Wire Line
+	5700 4350 5250 4350
+Wire Wire Line
+	4250 4450 4100 4450
+Wire Wire Line
+	4100 4450 4100 5900
+Wire Wire Line
+	4100 5900 4250 5900
+Wire Wire Line
+	4850 5900 4850 5250
+Connection ~ 4850 5250
+Wire Wire Line
+	4550 5900 4550 6250
+Wire Wire Line
+	4550 6250 5700 6250
+Wire Wire Line
+	5700 4350 5700 6250
+Connection ~ 4550 5900
 $EndSCHEMATC
